File: donkey-hat.kicad_pcb (KiCad board)
At the start: 2 copper layers, 65 x 56.5 mm, 65 parts, among them J1 6-18V, J14 NEOPIXEL, J15 MPU-9250, J16 4, J17 5, J18 6, J19 7, J2 Raspberry_Pi_2_3, J24 3mm_Mount, J25 3mm_Mount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

Commit message: Minor trace and silkscreen updates
Other:
- board text added: "Follow us: @mage0r @geekscape @jonoxer @thingc_co @heartofpluto_ @linuxaustralia @hackmelbourne"
- board text removed: "Follow us: @mage0r @geekscape @jonoxer @thingc @heartofpluto_ @linuxaustralia @hackmelbourne"
Changed lines of the file:
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@@
   )
   (setup
-    (last_trace_width 0.6)
+    (last_trace_width 0.15)
     (user_trace_width 0.15)
     (user_trace_width 0.2)
@@
     (effects (font (size 0.8 0.8) (thickness 0.15)) (justify mirror))
   )
-  (gr_text "Follow us:\n@mage0r\n@geekscape\n@jonoxer\n@thingc\n@heartofpluto_\n@linuxaustralia\n@hackmelbourne" (at 135.89 73.92) (layer B.SilkS)
+  (gr_text "Follow us:\n@mage0r\n@geekscape\n@jonoxer\n@thingc_co\n@heartofpluto_\n@linuxaustralia\n@hackmelbourne" (at 135.89 73.92) (layer B.SilkS)
     (effects (font (size 1 1) (thickness 0.15)) (justify left mirror))
   )

Commit message: Checking libs, project paths.
Parts:
- J1: footprint libs:ScrewTerminal-Small -> Connector_Phoenix_MC:PhoenixContact_MC_1,5_2-G-3.5_1x02_P3.50mm_Horizontal

Commit message: Remove ws2812. Keep header.
Parts:
- removed D2, D3: WS2812B, LED_SMD:LED_WS2812B_PLCC4_5.0x5.0mm_P3.2mm
Connections:
- J14 pad 2: /WS2812B_OUT -> /GPIO18
Routing:
- net Net-(D2-Pad2): track 34.7 -> 0.00 mm
- net /WS2812B_OUT: track 11.9 -> 0.00 mm
- net /GPIO18: track 45.8 -> 57.7 mm

Commit message: RM EEPROM.
Parts:
- removed JP1: WP, Jumper:SolderJumper-2_P1.3mm_Bridged_RoundedPad1.0x1.5mm
- removed R2: 3.9K, Resistor_SMD:R_0603_1608Metric_Pad1.05x0.95mm_HandSolder
- removed U1: CAT24C32, Package_SO:SOIC-8_3.9x4.9mm_P1.27mm
Changed lines of the file:
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@@
     (tracks 525)
     (zones 0)
-    (modules 63)
+    (modules 60)
     (nets 87)
   )
@@
     )
   )
-  (module Jumper:SolderJumper-2_P1.3mm_Bridged_RoundedPad1.0x1.5mm (layer F.Cu)
-    (at 128.46 75.96 270)
-    (descr "SMD Solder Jumper, 1x1.5mm, rounded Pads, 0.3mm gap, bridged with 1 copper strip")
-    (tags "solder jumper open")
-    (attr virtual)
-    (fp_text reference JP1 (at 0 -1.8 270) (layer F.SilkS) hide
-      (effects (font (size 1 1) (thickness 0.15)))
-    )
-    (fp_text value WP (at 2.37 0.01) (layer F.SilkS)
-      (effects (font (size 1 1) (thickness 0.15)))
-    )
-    (fp_arc (start 0.7 -0.3) (end 1.4 -0.3) (angle -90) (layer F.SilkS) (width 0.12))
-    (fp_arc (start 0.7 0.3) (end 0.7 1) (angle -90) (layer F.SilkS) (width 0.12))
-    (fp_arc (start -0.7 0.3) (end -1.4 0.3) (angle -90) (layer F.SilkS) (width 0.12))
-    (fp_arc (start -0.7 -0.3) (end -0.7 -1) (angle -90) (layer F.SilkS) (width 0.12))
-    (fp_line (start -1.4 0.3) (end -1.4 -0.3) (layer F.SilkS) (width 0.12))
-    (fp_line (start 0.7 1) (end -0.7 1) (layer F.SilkS) (width 0.12))
-    (fp_line (start 1.4 -0.3) (end 1.4 0.3) (layer F.SilkS) (width 0.12))
-    (fp_line (start -0.7 -1) (end 0.7 -1) (layer F.SilkS) (width 0.12))
-    (fp_line (start -1.65 -1.25) (end 1.65 -1.25) (layer F.CrtYd) (width 0.05))
-    (fp_line (start -1.65 -1.25) (end -1.65 1.25) (layer F.CrtYd) (width 0.05))
-    (fp_line (start 1.65 1.25) (end 1.65 -1.25) (layer F.CrtYd) (width 0.05))
-    (fp_line (start 1.65 1.25) (end -1.65 1.25) (layer F.CrtYd) (width 0.05))
-    (pad 1 smd custom (at -0.65 0 270) (size 1 0.5) (layers F.Cu F.Mask)
-      (net 61 "Net-(JP1-Pad1)") (zone_connect 0)
-      (options (clearance outline) (anchor rect))
-      (primitives
-        (gr_circle (center 0 0.25) (end 0.5 0.25) (width 0))
-        (gr_circle (center 0 -0.25) (end 0.5 -0.25) (width 0))
-        (gr_poly (pts
-           (xy 0 -0.75) (xy 0.5 -0.75) (xy 0.5 0.75) (xy 0 0.75)) (width 0))
-        (gr_poly (pts
-           (xy 0.9 -0.3) (xy 0.4 -0.3) (xy 0.4 0.3) (xy 0.9 0.3)) (width 0))
-      ))
-    (pad 2 smd custom (at 0.65 0 270) (size 1 0.5) (layers F.Cu F.Mask)
-      (net 1 GND) (zone_connect 0)
-      (options (clearance outline) (anchor rect))
-      (primitives
-        (gr_circle (center 0 0.25) (end 0.5 0.25) (width 0))
-        (gr_circle (center 0 -0.25) (end 0.5 -0.25) (width 0))
-        (gr_poly (pts
-           (xy 0 -0.75) (xy -0.5 -0.75) (xy -0.5 0.75) (xy 0 0.75)) (width 0))
-      ))
-  )
   (module Capacitor_SMD:C_0603_1608Metric_Pad1.05x0.95mm_HandSolder (layer F.Cu)
     (at 133.49 69.19 90)
@@
     )
   )
-  (module Package_SO:SOIC-8_3.9x4.9mm_P1.27mm (layer F.Cu)
-    (at 122.87 73.97)
-    (descr "8-Lead Plastic Small Outline (SN) - Narrow, 3.90 mm Body [SOIC] (see Microchip Packaging Specification 00000049BS.pdf)")
-    (tags "SOIC 1.27")
-    (attr smd)
-    (fp_text reference U1 (at 0 -3.5) (layer F.SilkS)
-      (effects (font (size 0.8 0.8) (thickness 0.15)))
-    )
-    (fp_text value CAT24C32 (at 0 3.5) (layer F.SilkS)
-      (effects (font (size 1 1) (thickness 0.15)))
-    )
-    (fp_text user %R (at 0 0) (layer F.Fab)
-      (effects (font (size 1 1) (thickness 0.15)))
-    )
-    (fp_line (start -0.95 -2.45) (end 1.95 -2.45) (layer F.Fab) (width 0.1))
-    (fp_line (start 1.95 -2.45) (end 1.95 2.45) (layer F.Fab) (width 0.1))
-    (fp_line (start 1.95 2.45) (end -1.95 2.45) (layer F.Fab) (width 0.1))
-    (fp_line (start -1.95 2.45) (end -1.95 -1.45) (layer F.Fab) (width 0.1))
-    (fp_line (start -1.95 -1.45) (end -0.95 -2.45) (layer F.Fab) (width 0.1))
-    (fp_line (start -3.73 -2.7) (end -3.73 2.7) (layer F.CrtYd) (width 0.05))
-    (fp_line (start 3.73 -2.7) (end 3.73 2.7) (layer F.CrtYd) (width 0.05))
-    (fp_line (start -3.73 -2.7) (end 3.73 -2.7) (layer F.CrtYd) (width 0.05))
-    (fp_line (start -3.73 2.7) (end 3.73 2.7) (layer F.CrtYd) (width 0.05))
-    (fp_line (start -2.075 -2.575) (end -2.075 -2.525) (layer F.SilkS) (width 0.15))
-    (fp_line (start 2.075 -2.575) (end 2.075 -2.43) (layer F.SilkS) (width 0.15))
-    (fp_line (start 2.075 2.575) (end 2.075 2.43) (layer F.SilkS) (width 0.15))
-    (fp_line (start -2.075 2.575) (end -2.075 2.43) (layer F.SilkS) (width 0.15))
-    (fp_line (start -2.075 -2.575) (end 2.075 -2.575) (layer F.SilkS) (width 0.15))
-    (fp_line (start -2.075 2.575) (end 2.075 2.575) (layer F.SilkS) (width 0.15))
-    (fp_line (start -2.075 -2.525) (end -3.475 -2.525) (layer F.SilkS) (width 0.15))
-    (pad 1 smd rect (at -2.7 -1.905) (size 1.55 0.6) (layers F.Cu F.Paste F.Mask)
-      (net 1 GND))
-    (pad 2 smd rect (at -2.7 -0.635) (size 1.55 0.6) (layers F.Cu F.Paste F.Mask)
-      (net 1 GND))
-    (pad 3 smd rect (at -2.7 0.635) (size 1.55 0.6) (layers F.Cu F.Paste F.Mask)
-      (net 1 GND))
-    (pad 4 smd rect (at -2.7 1.905) (size 1.55 0.6) (layers F.Cu F.Paste F.Mask)
-      (net 1 GND))
-    (pad 5 smd rect (at 2.7 1.905) (size 1.55 0.6) (layers F.Cu F.Paste F.Mask)
-      (net 45 /EEDATA))
-    (pad 6 smd rect (at 2.7 0.635) (size 1.55 0.6) (layers F.Cu F.Paste F.Mask)
-      (net 46 /EECLK))
-    (pad 7 smd rect (at 2.7 -0.635) (size 1.55 0.6) (layers F.Cu F.Paste F.Mask)
-      (net 61 "Net-(JP1-Pad1)"))
-    (pad 8 smd rect (at 2.7 -1.905) (size 1.55 0.6) (layers F.Cu F.Paste F.Mask)
-      (net 28 +3V3))
-    (model ${KISYS3DMOD}/Package_SO.3dshapes/SOIC-8_3.9x4.9mm_P1.27mm.wrl
-      (at (xyz 0 0 0))
-      (scale (xyz 1 1 1))
-      (rotate (xyz 0 0 0))
-    )
-  )
   (module Package_SO:TSSOP-28_4.4x9.7mm_P0.65mm (layer F.Cu)
     (at 103.2 100.07 90)
@@
     )
   )
-  (module Resistor_SMD:R_0603_1608Metric_Pad1.05x0.95mm_HandSolder (layer F.Cu)
-    (at 128.47 72.78 90)
-    (descr "Resistor SMD 0603 (1608 Metric), square (rectangular) end terminal, IPC_7351 nominal with elongated pad for handsoldering. (Body size source: http://www.tortai-tech.com/upload/download/2011102023233369053.pdf), generated with kicad-footprint-generator")
-    (tags "resistor handsolder")
-    (attr smd)
-    (fp_text reference R2 (at 2.29 0.01 180) (layer F.SilkS)
-      (effects (font (size 0.8 0.8) (thickness 0.15)))
-    )
-    (fp_text value 3.9K (at 0 1.43 90) (layer F.Fab) hide
-      (effects (font (size 1 1) (thickness 0.15)))
-    )
-    (fp_line (start -0.8 0.4) (end -0.8 -0.4) (layer F.Fab) (width 0.1))
-    (fp_line (start -0.8 -0.4) (end 0.8 -0.4) (layer F.Fab) (width 0.1))
-    (fp_line (start 0.8 -0.4) (end 0.8 0.4) (layer F.Fab) (width 0.1))
-    (fp_line (start 0.8 0.4) (end -0.8 0.4) (layer F.Fab) (width 0.1))
-    (fp_line (start -0.171267 -0.51) (end 0.171267 -0.51) (layer F.SilkS) (width 0.12))
-    (fp_line (start -0.171267 0.51) (end 0.171267 0.51) (layer F.SilkS) (width 0.12))
-    (fp_line (start -1.65 0.73) (end -1.65 -0.73) (layer F.CrtYd) (width 0.05))
-    (fp_line (start -1.65 -0.73) (end 1.65 -0.73) (layer F.CrtYd) (width 0.05))
-    (fp_line (start 1.65 -0.73) (end 1.65 0.73) (layer F.CrtYd) (width 0.05))
-    (fp_line (start 1.65 0.73) (end -1.65 0.73) (layer F.CrtYd) (width 0.05))
-    (fp_text user %R (at 0 0 90) (layer F.Fab)
-      (effects (font (size 0.4 0.4) (thickness 0.06)))
-    )
-    (pad 1 smd roundrect (at -0.875 0 90) (size 1.05 0.95) (layers F.Cu F.Paste F.Mask) (roundrect_rratio 0.25)
-      (net 61 "Net-(JP1-Pad1)"))
-    (pad 2 smd roundrect (at 0.875 0 90) (size 1.05 0.95) (layers F.Cu F.Paste F.Mask) (roundrect_rratio 0.25)
-      (net 28 +3V3))
-    (model ${KISYS3DMOD}/Resistor_SMD.3dshapes/R_0603_1608Metric.wrl
-      (at (xyz 0 0 0))
-      (scale (xyz 1 1 1))
-      (rotate (xyz 0 0 0))
-    )
-  )
   (module Capacitor_SMD:C_0603_1608Metric_Pad1.05x0.95mm_HandSolder (layer F.Cu)
     (at 133.81 108.48 90)
@@
   (segment (start 84.47 79.99) (end 84.47 97.568786) (width 1) (layer B.Cu) (net 2))
   (segment (start 84.47 97.568786) (end 83.358786 98.68) (width 1) (layer B.Cu) (net 2))
-  (segment (start 139.53 108.17) (end 136.4 111.3) (width 0.25) (layer F.Cu) (net 34))
-  (segment (start 140.28 108.17) (end 139.53 108.17) (width 0.25) (layer F.Cu) (net 34))
-  (segment (start 132.81 111.3) (end 130.59 113.52) (width 0.25) (layer F.Cu) (net 34))
-  (segment (start 136.4 111.3) (end 132.81 111.3) (width 0.25) (layer F.Cu) (net 34))
   (segment (start 117.51 97.18) (end 118.01 97.18) (width 0.25) (layer F.Cu) (net 3) (status 20))
   (segment (start 117.17 97.18) (end 117.51 97.18) (width 0.25) (layer F.Cu) (net 3))
@@
   (segment (start 81.625 107.75) (end 81.605 107.73) (width 0.25) (layer F.Cu) (net 29) (status 30))
   (segment (start 83.545 107.75) (end 81.625 107.75) (width 0.25) (layer F.Cu) (net 29) (status 30))
+  (segment (start 139.53 108.17) (end 136.4 111.3) (width 0.25) (layer F.Cu) (net 34))
+  (segment (start 140.28 108.17) (end 139.53 108.17) (width 0.25) (layer F.Cu) (net 34))
+  (segment (start 132.81 111.3) (end 130.59 113.52) (width 0.25) (layer F.Cu) (net 34))
+  (segment (start 136.4 111.3) (end 132.81 111.3) (width 0.25) (layer F.Cu) (net 34))
   (segment (start 99.62 63.05) (end 101.19 61.48) (width 0.25) (layer F.Cu) (net 34))
   (segment (start 101.19 61.48) (end 135.9 61.48) (width 0.25) (layer F.Cu) (net 34))
