File: dingo-hat.sch (KiCad schematic (older format))
At the start: 54 parts, among them J1 6-18V, J14 NEOPIXEL, J15 MPU-9250, J16 4, J17 5, J18 6, J19 7, J2 Raspberry_Pi_2_3, J24 3mm_Mount, J25 3mm_Mount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

Commit message: Adding schematic library for graphics/logos.
Parts:
- added G?: LCA2020Logo, symbol graphics:LCA2020Logo
- added G?: CCHSLogo, symbol graphics:CCHSLogo
Other:
- note added: "Graphics/Logos"
Changed lines of the file:
@@
 EESchema Schematic File Version 4
-LIBS:donkey-hat-cache
+LIBS:dingo-hat-cache
 EELAYER 30 0
 EELAYER END
@@
 Text Notes 4600 7350 0    118  ~ 24
 Add some I/O protection.
+$Comp
+L graphics:LCA2020Logo G?
+U 1 1 5DA95D6D
+P 600 7200
+F 0 "G?" H 550 7200 50  0000 L CNN
+F 1 "LCA2020Logo" H 600 7200 50  0001 C CNN
+F 2 "" H 600 7200 50  0001 C CNN
+F 3 "" H 600 7200 50  0001 C CNN
+	1    600  7200
+	1    0    0    -1
+$EndComp
+$Comp
+L graphics:CCHSLogo G?
+U 1 1 5DA9B14E
+P 600 7100
+F 0 "G?" H 550 7100 50  0000 L CNN
+F 1 "CCHSLogo" H 600 7100 50  0001 C CNN
+F 2 "" H 600 7100 50  0001 C CNN
+F 3 "" H 600 7100 50  0001 C CNN
+	1    600  7100
+	1    0    0    -1
+$EndComp
+Wire Notes Line
+	1150 7800 1150 6850
+Wire Notes Line
+	1150 6850 500  6850
+Text Notes 450  6950 0    50   ~ 0
+Graphics/Logos
 $EndSCHEMATC
